Commit message: Added new URDF

File: data/assets/urdf/hh_hand.urdf (robot description, URDF)
Before this commit: robot converted_robot, 99 links, 98 joints
Links:
- removed link index_pp2index_pp_sens_fixed_jointbody
- removed link index_pp_sens
- removed link middle_pp2middle_pp_sens_fixed_jointbody
- removed link middle_pp_sens
- removed link ring_pp2ring_pp_sens_fixed_jointbody
- removed link ring_pp_sens
- link index_dp: mass 0.0014084542990363813 -> 0.00548455016800106
- link middle_dp: mass 0.0014084542990363813 -> 0.00548455016800106
- link pinky_dp: mass 0.0014084542990363813 -> 0.00548455016800106
- link ring_dp: mass 0.0014084542990363813 -> 0.00548455016800106
- link root: mass 1.7061285524984284 -> 1.2601437096752013
- link thumb_dp: mass 0.003041625293114536 -> 0.00548455016800106
Joints:
- removed joint index_pp2index_pp_sens_fixed
- removed joint index_pp2index_pp_sens_fixed_offset
- removed joint middle_pp2middle_pp_sens_fixed
- removed joint middle_pp2middle_pp_sens_fixed_offset
- removed joint ring_pp2ring_pp_sens_fixed
- removed joint ring_pp2ring_pp_sens_fixed_offset
- joint index_dp2index_fingertip_fixed: origin xyz=0.0 0.0 0.01 rpy=0.0 0.0 0.0 -> xyz=0.02 0.0 0.0 rpy=0.0 0.0 0.0
- joint middle_dp2middle_fingertip_fixed: origin xyz=0.0 0.0 0.01 rpy=0.0 0.0 0.0 -> xyz=0.02 0.0 0.0 rpy=0.0 0.0 0.0
- joint pinky_dp2pinky_fingertip_fixed: origin xyz=0.0 0.0 0.01 rpy=0.0 0.0 0.0 -> xyz=0.02 0.0 0.0 rpy=0.0 0.0 0.0
- joint ring_dp2ring_fingertip_fixed: origin xyz=0.0 0.0 0.01 rpy=0.0 0.0 0.0 -> xyz=0.02 0.0 0.0 rpy=0.0 0.0 0.0
- joint root2thumb_base: limit lower=-0.349 upper=2.094 effort=100 velocity=100 -> lower=0.0 upper=2.356 effort=100 velocity=100
- joint thumb_dp2thumb_fingertip_fixed: origin xyz=0.000386 -0.000394 -0.012633 rpy=1.583092548356868 0.21851142430155246 -2.8889085939445414 -> xyz=0.02 0.0 0.0 rpy=0.0 0.0 0.0

Commit message: Fixed thumb URDF visualization

File: data/assets/urdf/hh_hand.urdf (robot description, URDF)
Before this commit: robot converted_robot, 93 links, 92 joints
Links:
- removed link pinky_pp2pinky_pp_sens_fixed_jointbody
- removed link pinky_pp_sens
Joints:
- removed joint pinky_pp2pinky_pp_sens_fixed
- removed joint pinky_pp2pinky_pp_sens_fixed_offset
- joint thumb_base2pp: limit lower=-0.785 upper=0.785 effort=100 velocity=100 -> lower=0.0 upper=1.48 effort=100 velocity=100; origin xyz=0.006722907138596131 0.0007866772718234209 0.007535891827401083 rpy=-1.5649041390916683 0.7831397689767283 -0.8634482425952612 -> xyz=0.006533598964040238 0.0009856559418268736 0.007298535710728157 rpy=-1.5522799247268875 0.7886936673883342 -1.5522799247268875

Commit message: Improvements to thumb retargetting

File: data/assets/urdf/hh_hand.urdf (robot description, URDF)
Before this commit: robot converted_robot, 91 links, 90 joints
Links:
- link thumb_dp: mass 0.00548455016800106 -> 0.007138375295193356
Joints:
- joint thumb_dp2thumb_fingertip_fixed: origin xyz=0.02 0.0 0.0 rpy=0.0 0.0 0.0 -> xyz=0.03 0.0 0.0 rpy=0.0 0.0 0.0

Commit message: Added knuckle keyvectors and palm translation

File: data/assets/urdf/hh_hand.urdf (robot description, URDF)
Before this commit: robot converted_robot, 91 links, 90 joints
Links:
- added link retarget_palm, mass 0.001
Joints:
- added joint retarget_palm_offset: type fixed, parent palm, child retarget_palm, origin xyz=-0.015 0.00 0 rpy=0 0 0
